Commit message: Fix and tune gazebo simulation
Use dynamic reconfigure for PID parameters
Publish unactuated joint states

File: robotiq_2f_85_gripper_visualization/urdf/gazebo.urdf.xacro (robot description, xacro)
@@ -1,8 +1,9 @@
 <?xml version="1.0"?>
-<robot xmlns:xacro="http://ros.org/wiki/xacro">
+<robot xmlns:xacro="http://www.ros.org/wiki/xacro">
   <gazebo>
     <plugin name="robotiq2f" filename="libRobotiq2fPlugin.so">
         <loop_joint name="left_loop_joint" parent="left_knuckle_dummy_link" child="left_inner_finger"/>
         <loop_joint name="right_loop_joint" parent="right_knuckle_dummy_link" child="right_inner_finger"/>
+        <joint_states>/robot/joint_states</joint_states>
     </plugin>
     <plugin name="mimic_joint" filename="libroboticsgroup_gazebo_mimic_joint_plugin.so">
@@ -12,4 +13,5 @@
     </plugin>
   </gazebo>
+<!--
   <link name="world"/>
   <joint name="fixingModelInPlace" type="fixed">
@@ -18,3 +20,4 @@
       <child link="robotiq_arg2f_base_link" />
   </joint>
+-->
 </robot>

File: robotiq_2f_85_gripper_visualization/urdf/robotiq_arg2f.xacro (robot description, xacro)
@@ -1,4 +1,4 @@
 <?xml version="1.0"?>
-<robot xmlns:xacro="http://ros.org/wiki/xacro">
+<robot xmlns:xacro="http://www.ros.org/wiki/xacro">
   <xacro:macro name="robotiq_arg2f_base_link" params="prefix">
     <link name="${prefix}robotiq_arg2f_base_link">

File: robotiq_2f_85_gripper_visualization/urdf/robotiq_arg2f_85_model.xacro (robot description, xacro)
@@ -1,4 +1,4 @@
 <?xml version="1.0"?>
-<robot name="robotiq_arg2f_85_model" xmlns:xacro="http://ros.org/wiki/xacro">
+<robot name="robotiq_arg2f_85_model" xmlns:xacro="http://www.ros.org/wiki/xacro">
   <xacro:include filename="$(find robotiq_2f_85_gripper_visualization)/urdf/robotiq_arg2f_85_model_macro.xacro" />
   <xacro:include filename="$(find robotiq_2f_85_gripper_visualization)/urdf/gazebo.urdf.xacro"/>

File: robotiq_2f_85_gripper_visualization/urdf/robotiq_arg2f_85_model_macro.xacro (robot description, xacro)
@@ -1,5 +1,5 @@
 <?xml version="1.0"?>
-<robot xmlns:xacro="http://ros.org/wiki/xacro">
-  <xacro:include filename="$(find robotiq_2f_85_gripper_visualization)/urdf/robotiq_arg2f_transmission.xacro" />
+<robot xmlns:xacro="http://www.ros.org/wiki/xacro">
+<!--  <xacro:include filename="$(find robotiq_2f_85_gripper_visualization)/urdf/robotiq_arg2f_transmission.xacro" /> -->
   <xacro:macro name="outer_knuckle" params="prefix fingerprefix stroke">
     <link name="${prefix}${fingerprefix}_outer_knuckle">
@@ -136,5 +136,5 @@
       <child link="${prefix}${fingerprefix}_inner_knuckle" />
       <axis xyz="1 0 0" />
-      <limit lower="0" upper="1.0" velocity="2.0" effort="1000" />
+      <limit lower="0" upper="1.0" velocity="2.0" effort="220" />
       <mimic joint="${prefix}finger_joint" multiplier="1" offset="0" />
    </joint>
@@ -167,5 +167,5 @@
       <child link="${prefix}${fingerprefix}_knuckle_dummy_link" />
       <axis xyz="1 0 0" />
-      <limit lower="-3.14" upper="3.14" velocity="2.0" effort="1000" />
+      <limit lower="-3.14" upper="3.14" velocity="2.0" effort="220" />
     </joint>
   </xacro:macro>
@@ -176,5 +176,5 @@
       <child link="${prefix}${fingerprefix}_inner_finger" />
       <axis xyz="1 0 0" />
-      <limit lower="-3.14" upper="3.14" velocity="2.0" effort="1000" />
+      <limit lower="-3.14" upper="3.14" velocity="2.0" effort="220" />
       <mimic joint="${prefix}finger_joint" multiplier="-1" offset="0" />
     </joint>
@@ -195,7 +195,5 @@
       <child link="${prefix}left_outer_knuckle" />
       <axis xyz="1 0 0" />
-      <limit lower="0" upper="0.8" velocity="2.0" effort="1000" />
-      <position_effort_min>-1</position_effort_min>
-      <position_effort_max>1</position_effort_max>
+      <limit lower="0" upper="0.8" velocity="2.0" effort="220" />
     </joint>
     <xacro:finger_joints prefix="${prefix}" fingerprefix="left" reflect="1.0"/>
@@ -207,5 +205,5 @@
       <child link="${prefix}right_outer_knuckle" />
       <axis xyz="1 0 0" />
-      <limit lower="0" upper="0.81" velocity="2.0" effort="1000" />
+      <limit lower="0" upper="0.81" velocity="2.0" effort="220" />
       <mimic joint="${prefix}finger_joint" multiplier="1" offset="0" />
     </joint>
@@ -219,5 +217,5 @@
     <xacro:finger_joint prefix="${prefix}"/>
     <xacro:right_outer_knuckle_joint prefix="${prefix}"/>
-    <xacro:robotiq_arg2f_transmission prefix="${prefix}"/>
+<!--    <xacro:robotiq_arg2f_transmission prefix="${prefix}"/>-->
   </xacro:macro>
 </robot>

File: robotiq_2f_85_gripper_visualization/urdf/robotiq_arg2f_transmission.xacro (robot description, xacro)
@@ -1,4 +1,4 @@
 <?xml version="1.0"?>
-<robot xmlns:xacro="http://ros.org/wiki/xacro">
+<robot xmlns:xacro="http://www.ros.org/wiki/xacro">
   <xacro:macro name="robotiq_arg2f_transmission" params="prefix">
     <transmission name="${prefix}finger_joint_trans">
