Commit message: test recursive push robotiq

File: robotiq_2f_85_gripper_visualization/urdf/robotiq_arg2f_85_model_macro.xacro (robot description, xacro)
@@ -6,5 +6,6 @@
       <inertial>
         <origin xyz="-0.000200000000003065 0.0199435877845359 0.0292245259211331" rpy="0 0 0" />
-        <mass value="0.00853198276973456" />
+        <!-- <mass value="0.00853198276973456" /> -->
+        <mass value="2.89328108496468E-06" />
         <inertia ixx="2.89328108496468E-06" ixy="-1.57935047237397E-19" ixz="-1.93980378593255E-19" iyy="1.86719750325683E-06" iyz="-1.21858577871576E-06" izz="1.21905238907251E-06" />
         </inertial>
@@ -30,5 +31,6 @@
       <inertial>
         <origin xyz="0.00030115855001899 0.0373907951953854 -0.0208027427000385" rpy="0 0 0" />
-        <mass value="0.022614240507152" />
+        <!-- <mass value="0.022614240507152" /> -->
+        <mass value="1.52518312458174E-05" />
         <inertia ixx="1.52518312458174E-05" ixy="9.76583423954399E-10" ixz="-5.43838577022588E-10" iyy="6.17694243867776E-06" iyz="6.78636130740228E-06" izz="1.16494917907219E-05" />
         </inertial>
@@ -54,5 +56,6 @@
       <inertial>
         <origin xyz="0.000123011831763771 0.0507850843201817 0.00103968640075166" rpy="0 0 0" />
-       <mass value="0.0271177346495152" />
+       <!-- <mass value="0.0271177346495152" /> -->
+       <mass value="2.61910379223783E-05" />
         <inertia ixx="2.61910379223783E-05" ixy="-2.43616858946494E-07" ixz="-6.37789906117123E-09" iyy="2.8270243746167E-06" iyz="-5.37200748039765E-07" izz="2.83695868220296E-05" />
         </inertial>
@@ -78,5 +81,6 @@
       <inertial>
         <origin xyz="0.000299999999999317 0.0160078233491243 -0.0136945669206257" rpy="0 0 0" />
-        <mass value="0.0104003125914103" />
+        <!-- <mass value="0.0104003125914103" /> -->
+        <mass value="2.71909453810972E-06" />
         <inertia ixx="2.71909453810972E-06" ixy="1.35402465472579E-21" ixz="-7.1817349065269E-22" iyy="7.69100314106116E-07" iyz="6.74715432769696E-07" izz="2.30315190420171E-06" />
         </inertial>
@@ -142,5 +146,6 @@
       <inertial>
         <origin xyz="0 0 0" rpy="0 0 0" />
-       <mass value="0.001" />
+       <!-- <mass value="0.001" /> -->
+       <mass value="2.61910379223783E-05" />
         <inertia ixx="2.61910379223783E-05" ixy="-2.43616858946494E-07" ixz="-6.37789906117123E-09" iyy="2.8270243746167E-06" iyz="-5.37200748039765E-07" izz="2.83695868220296E-05" />
         </inertial>

Commit message: updating gripper xacro

File: robotiq_2f_85_gripper_visualization/urdf/robotiq_arg2f_85_model_macro.xacro (robot description, xacro)
@@ -6,6 +6,5 @@
       <inertial>
         <origin xyz="-0.000200000000003065 0.0199435877845359 0.0292245259211331" rpy="0 0 0" />
-        <!-- <mass value="0.00853198276973456" /> -->
-        <mass value="2.89328108496468E-06" />
+        <mass value="0.00853198276973456" />
         <inertia ixx="2.89328108496468E-06" ixy="-1.57935047237397E-19" ixz="-1.93980378593255E-19" iyy="1.86719750325683E-06" iyz="-1.21858577871576E-06" izz="1.21905238907251E-06" />
         </inertial>
@@ -31,6 +30,5 @@
       <inertial>
         <origin xyz="0.00030115855001899 0.0373907951953854 -0.0208027427000385" rpy="0 0 0" />
-        <!-- <mass value="0.022614240507152" /> -->
-        <mass value="1.52518312458174E-05" />
+        <mass value="0.022614240507152" />
         <inertia ixx="1.52518312458174E-05" ixy="9.76583423954399E-10" ixz="-5.43838577022588E-10" iyy="6.17694243867776E-06" iyz="6.78636130740228E-06" izz="1.16494917907219E-05" />
         </inertial>
@@ -56,6 +54,5 @@
       <inertial>
         <origin xyz="0.000123011831763771 0.0507850843201817 0.00103968640075166" rpy="0 0 0" />
-       <!-- <mass value="0.0271177346495152" /> -->
-       <mass value="2.61910379223783E-05" />
+       <mass value="0.0271177346495152" />
         <inertia ixx="2.61910379223783E-05" ixy="-2.43616858946494E-07" ixz="-6.37789906117123E-09" iyy="2.8270243746167E-06" iyz="-5.37200748039765E-07" izz="2.83695868220296E-05" />
         </inertial>
@@ -81,6 +78,5 @@
       <inertial>
         <origin xyz="0.000299999999999317 0.0160078233491243 -0.0136945669206257" rpy="0 0 0" />
-        <!-- <mass value="0.0104003125914103" /> -->
-        <mass value="2.71909453810972E-06" />
+        <mass value="0.0104003125914103" />
         <inertia ixx="2.71909453810972E-06" ixy="1.35402465472579E-21" ixz="-7.1817349065269E-22" iyy="7.69100314106116E-07" iyz="6.74715432769696E-07" izz="2.30315190420171E-06" />
         </inertial>
@@ -146,6 +142,5 @@
       <inertial>
         <origin xyz="0 0 0" rpy="0 0 0" />
-       <!-- <mass value="0.001" /> -->
-       <mass value="2.61910379223783E-05" />
+       <mass value="0.001" />
         <inertia ixx="2.61910379223783E-05" ixy="-2.43616858946494E-07" ixz="-6.37789906117123E-09" iyy="2.8270243746167E-06" iyz="-5.37200748039765E-07" izz="2.83695868220296E-05" />
         </inertial>
